Commit message: Add files via upload

File: t1_rover/urdf/leo_sim.urdf.xacro (robot description, xacro)
@@ -3,9 +3,7 @@
        name="leo_sim">
   <xacro:arg name="fixed" default="false"/>
-  <xacro:arg name="robot_ns" default=""/>
   <xacro:arg name="mecanum_wheels" default="false"/>
-  <xacro:include filename="$(find t1_rover)/urdf/macros.xacro"/>
-  <xacro:leo_sim robot_ns="$(arg robot_ns)"
-                 fixed="$(arg fixed)"
+  <xacro:include filename="$(find t1_rover)/urdf/macros2.xacro"/>
+  <xacro:leo_sim fixed="$(arg fixed)"
                  mecanum_wheels="$(arg mecanum_wheels)"/>
 </robot>

File: t1_rover/urdf/macros.xacro (robot description, xacro)
@@ -1,17 +1,12 @@
 <?xml version="1.0" encoding="utf-8"?>
 <robot xmlns:xacro="http://www.ros.org/wiki/xacro">
-  <xacro:property name="package_name" value="t1_rover" />
   <xacro:macro name="leo"
                params="default_antenna:=true
                        rockers_fixed:=true
                        footprint_link:=true
-                       link_prefix:=''
-                       joint_prefix:=''
                        imu_translation:='0.0628 -0.0314 -0.0393'
                        mecanum_wheels:=false">
-    <!-- Include and namespace the laser component -->
-    <xacro:include filename="$(find t1_rover)/urdf/laser.xacro"/>
     <xacro:macro name="rocker_link" params="name">
-      <link name="${link_prefix}rocker_${name}_link">
+      <link name="rocker_${name}_link">
         <inertial>
           <mass value="1.387336"/>
@@ -35,5 +30,5 @@
     </xacro:macro>
     <xacro:macro name="wheel_link" params="name model">
-      <link name="${link_prefix}wheel_${name}_link">
+      <link name="wheel_${name}_link">
         <inertial>
           <mass value="0.283642"/>
@@ -69,5 +64,5 @@
     </xacro:macro>
     <xacro:macro name="mecanum_wheel_link" params="name model">
-      <link name="${link_prefix}wheel_${name}_link">
+      <link name="wheel_${name}_link">
         <inertial>
           <mass value="0.672214"/>
@@ -98,7 +93,7 @@
     <!-- LINKS -->
     <xacro:if value="${footprint_link}">
-      <link name="${link_prefix}base_footprint"/>
-    </xacro:if>
-    <link name="${link_prefix}base_link">
+      <link name="base_footprint"/>
+    </xacro:if>
+    <link name="base_link">
       <inertial>
         <mass value="1.584994"/>
@@ -135,5 +130,5 @@
     </xacro:unless>
     <xacro:if value="${default_antenna}">
-      <link name="${link_prefix}antenna_link">
+      <link name="antenna_link">
         <inertial>
           <mass value="0.001237"/>
@@ -157,13 +152,47 @@
       </link>
     </xacro:if>
-    <link name="${link_prefix}camera_frame"/>
-    <link name="${link_prefix}camera_optical_frame"/>
-    <link name="${link_prefix}imu_frame"/>
+    <link name="camera_frame"/>
+    <link name="camera_optical_frame"/>
+    <link name="imu_frame"/>
+    <link name="laser_frame"/>
+    <!--LIDAR LINK-->
+    <link name="rplidar_link">
+    <visual>
+      <origin xyz="0 0 0.003"/>
+      <geometry>
+        <box size="0.079 0.086 0.006"/>
+      </geometry>
+      <material name="support">
+        <color rgba="0.5 0.5 0.5 1.0"/>
+      </material>
+    </visual>
+    <visual>
+      <origin xyz="0 0 0.023"/>
+      <geometry>
+        <cylinder radius="0.038" length="0.04"/>
+      </geometry>
+      <material name="lidar">
+        <color rgba="1.0 0.0 0.0 0.7"/>
+      </material>
+    </visual>
+    <collision>
+      <origin xyz="0 0 0.003"/>
+      <geometry>
+        <box size="0.079 0.086 0.006"/>
+      </geometry>
+    </collision>
+    <collision>
+      <origin xyz="0 0 0.023"/>
+      <geometry>
+        <cylinder radius="0.038" length="0.04"/>
+      </geometry>
+    </collision>
+  </link>
     <!-- JOINTS -->
     <xacro:if value="${footprint_link}">
-      <joint name="${joint_prefix}base_joint" type="fixed">
+      <joint name="base_joint" type="fixed">
         <origin xyz="0 0 0.19783" rpy="0 0 0"/>
-        <parent link="${link_prefix}base_footprint"/>
-        <child link="${link_prefix}base_link"/>
+        <parent link="base_footprint"/>
+        <child link="base_link"/>
       </joint>
     </xacro:if>
@@ -174,16 +203,16 @@
       <xacro:property name="rockers_joint_type" value="revolute"/>
     </xacro:unless>
-    <joint name="${joint_prefix}rocker_L_joint" type="${rockers_joint_type}">
+    <joint name="rocker_L_joint" type="${rockers_joint_type}">
       <origin xyz="0.00263 0.14167 -0.04731" rpy="0 0 ${pi}"/>
-      <parent link="${link_prefix}base_link"/>
-      <child link="${link_prefix}rocker_L_link"/>
+      <parent link="base_link"/>
+      <child link="rocker_L_link"/>
       <axis xyz="0 1 0"/>
       <limit effort="100.0" lower="-0.24" upper="0.24" velocity="100.0"/>
       <dynamics friction="1.0" damping="0.1"/>
     </joint>
-    <joint name="${joint_prefix}rocker_R_joint" type="${rockers_joint_type}">
+    <joint name="rocker_R_joint" type="${rockers_joint_type}">
       <origin xyz="0.00263 -0.14167 -0.04731" rpy="0 0 0"/>
-      <parent link="${link_prefix}base_link"/>
-      <child link="${link_prefix}rocker_R_link"/>
+      <parent link="base_link"/>
+      <child link="rocker_R_link"/>
       <axis xyz="0 1 0"/>
       <limit effort="100.0" lower="-0.24" upper="0.24" velocity="100.0"/>
@@ -191,5 +220,5 @@
       <mimic joint="rocker_L_joint"/>
     </joint>
-    <joint name="${joint_prefix}wheel_FL_joint" type="continuous">
+    <joint name="wheel_FL_joint" type="continuous">
       <xacro:if value="${mecanum_wheels}">
         <origin xyz="-0.15256 -0.00884 -0.08802" rpy="0 0 0"/>
@@ -198,11 +227,11 @@
         <origin xyz="-0.15256 -0.08214 -0.08802" rpy="0 0 0"/>
       </xacro:unless>
-      <parent link="${link_prefix}rocker_L_link"/>
-      <child link="${link_prefix}wheel_FL_link"/>
+      <parent link="rocker_L_link"/>
+      <child link="wheel_FL_link"/>
       <axis xyz="0 -1 0"/>
       <limit effort="2.0" velocity="6.0"/>
       <dynamics friction="0.3125" damping="0.1"/>
     </joint>
-    <joint name="${joint_prefix}wheel_RL_joint" type="continuous">
+    <joint name="wheel_RL_joint" type="continuous">
       <xacro:if value="${mecanum_wheels}">
         <origin xyz="0.15256 -0.00884 -0.08802" rpy="0 0 0"/>
@@ -211,11 +240,11 @@
         <origin xyz="0.15256 -0.08214 -0.08802" rpy="0 0 0"/>
       </xacro:unless>
-      <parent link="${link_prefix}rocker_L_link"/>
-      <child link="${link_prefix}wheel_RL_link"/>
+      <parent link="rocker_L_link"/>
+      <child link="wheel_RL_link"/>
       <axis xyz="0 -1 0"/>
       <limit effort="2.0" velocity="6.0"/>
       <dynamics friction="0.3125" damping="0.1"/>
     </joint>
-    <joint name="${joint_prefix}wheel_FR_joint" type="continuous">
+    <joint name="wheel_FR_joint" type="continuous">
       <xacro:if value="${mecanum_wheels}">
         <origin xyz="0.15256 -0.00884 -0.08802" rpy="0 0 0"/>
@@ -224,11 +253,11 @@
         <origin xyz="0.15256 -0.08214 -0.08802" rpy="0 0 0"/>
       </xacro:unless>
-      <parent link="${link_prefix}rocker_R_link"/>
-      <child link="${link_prefix}wheel_FR_link"/>
+      <parent link="rocker_R_link"/>
+      <child link="wheel_FR_link"/>
       <axis xyz="0 1 0"/>
       <limit effort="2.0" velocity="6.0"/>
       <dynamics friction="0.3125" damping="0.1"/>
     </joint>
-    <joint name="${joint_prefix}wheel_RR_joint" type="continuous">
+    <joint name="wheel_RR_joint" type="continuous">
       <xacro:if value="${mecanum_wheels}">
         <origin xyz="-0.15256 -0.00884 -0.08802" rpy="0 0 0"/>
@@ -237,6 +266,6 @@
         <origin xyz="-0.15256 -0.08214 -0.08802" rpy="0 0 0"/>
       </xacro:unless>
-      <parent link="${link_prefix}rocker_R_link"/>
-      <child link="${link_prefix}wheel_RR_link"/>
+      <parent link="rocker_R_link"/>
+      <child link="wheel_RR_link"/>
       <axis xyz="0 1 0"/>
       <limit effort="2.0" velocity="6.0"/>
@@ -244,35 +273,40 @@
     </joint>
     <xacro:if value="${default_antenna}">
-      <joint name="${joint_prefix}antenna_joint" type="fixed">
+      <joint name="antenna_joint" type="fixed">
         <origin xyz="-0.0052 0.056 -0.0065" rpy="0 0 0"/>
-        <parent link="${link_prefix}base_link"/>
-        <child link="${link_prefix}antenna_link"/>
+        <parent link="base_link"/>
+        <child link="antenna_link"/>
       </joint>
     </xacro:if>
-    <joint name="${joint_prefix}camera_joint" type="fixed">
+    <joint name="camera_joint" type="fixed">
       <origin xyz="0.0971 0 -0.0427" rpy="0 0.2094 0"/>
-      <parent link="${link_prefix}base_link"/>
-      <child link="${link_prefix}camera_frame"/>
-    </joint>
-    <joint name="${joint_prefix}camera_optical_joint" type="fixed">
+      <parent link="base_link"/>
+      <child link="camera_frame"/>
+    </joint>
+    <joint name="camera_optical_joint" type="fixed">
       <origin xyz="0 0 0" rpy="-${pi/2} 0.0 -${pi/2}"/>
-      <parent link="${link_prefix}camera_frame"/>
-      <child link="${link_prefix}camera_optical_frame"/>
-    </joint>
-    <joint name="${joint_prefix}imu_joint" type="fixed">
+      <parent link="camera_frame"/>
+      <child link="camera_optical_frame"/>
+    </joint>
+    <joint name="imu_joint" type="fixed">
       <origin xyz="${imu_translation}" rpy="0 0 0"/>
-      <parent link="${link_prefix}base_link"/>
-      <child link="${link_prefix}imu_frame"/>
+      <parent link="base_link"/>
+      <child link="imu_frame"/>
+    </joint>
+    <joint name="rplidar_joint" type="fixed">
+      <origin xyz="0.0775 0 0"/>
+      <parent link="base_link"/>
+      <child link="rplidar_link"/>
+    </joint>
+    <joint name="laser_joint" type="fixed">
+      <origin xyz="0 0 0.0368" rpy="0 0 ${pi}"/>
+      <parent link="rplidar_link"/>
+      <child link="laser_frame"/>
     </joint>
   </xacro:macro>
   <!-- LEO GAZEBO -->
-  <xacro:macro name="leo_gazebo"
-               params="robot_ns:='''">
-    <xacro:property name="link_prefix" value=""/>
-    <xacro:if value="${robot_ns != '' and robot_ns != '/'}">
-      <xacro:property name="link_prefix" value="${robot_ns}/"/>
-    </xacro:if>
+  <xacro:macro name="leo_gazebo">
     <!-- base ODE properties -->
-    <gazebo reference="${link_prefix}base_footprint">
+    <gazebo reference="base_footprint">
       <collision>
         <surface>
@@ -291,5 +325,5 @@
       </collision>
     </gazebo>
-    <gazebo reference="${link_prefix}base_link">
+    <gazebo reference="base_link">
       <collision>
         <surface>
@@ -309,5 +343,5 @@
     </gazebo>
     <!-- rocker ODE properties -->
-    <gazebo reference="${link_prefix}rocker_L_link">
+    <gazebo reference="rocker_L_link">
       <collision>
         <surface>
@@ -326,5 +360,5 @@
       </collision>
     </gazebo>
-    <gazebo reference="${link_prefix}rocker_R_link">
+    <gazebo reference="rocker_R_link">
       <collision>
         <surface>
@@ -344,5 +378,5 @@
     </gazebo>
     <!-- wheel ODE properties -->
-    <gazebo reference="${link_prefix}wheel_FL_link">
+    <gazebo reference="wheel_FL_link">
       <collision>
         <surface>
@@ -364,5 +398,5 @@
       </collision>
     </gazebo>
-    <gazebo reference="${link_prefix}wheel_FR_link">
+    <gazebo reference="wheel_FR_link">
       <collision>
         <surface>
@@ -384,5 +418,5 @@
       </collision>
     </gazebo>
-    <gazebo reference="${link_prefix}wheel_RL_link">
+    <gazebo reference="wheel_RL_link">
       <collision>
         <surface>
@@ -404,5 +438,5 @@
       </collision>
     </gazebo>
-    <gazebo reference="${link_prefix}wheel_RR_link">
+    <gazebo reference="wheel_RR_link">
       <collision>
         <surface>
@@ -425,5 +459,5 @@
     </gazebo>
     <!-- camera -->
-    <gazebo reference="${link_prefix}camera_frame">
+    <gazebo reference="camera_frame">
       <sensor name="camera" type="camera">
           <camera name="leo_camera">
@@ -455,12 +489,61 @@
           <update_rate>30</update_rate>
           <visualize>true</visualize>
-          <topic>${link_prefix}camera/image_raw</topic>
-          <ignition_frame_id>${link_prefix}camera_frame</ignition_frame_id>
+          <topic>camera/image_raw</topic>
+          <ignition_frame_id>camera_frame</ignition_frame_id>
       </sensor>
     </gazebo>
-    <!-- lidar -->
+    <!-- rocker differential -->
+    <gazebo>
+      <plugin name="leo_gz::DifferentialSystem" filename="libleo_gz_differential_plugin.so">
+        <jointA>rocker_L_joint</jointA>
+        <jointB>rocker_R_joint</jointB>
+        <forceConstant>100.0</forceConstant>
+      </plugin>
+    </gazebo>
+    <gazebo>
+      <plugin
+        filename="ignition-gazebo-joint-state-publisher-system"
+        name="ignition::gazebo::systems::JointStatePublisher">
+        <topic>joint_states</topic>
+      </plugin>
+      <plugin filename="libignition-gazebo-imu-system.so"
+        name="ignition::gazebo::systems::Imu">
+      </plugin>
+    </gazebo>
+    <gazebo reference="imu_frame">
+      <sensor type="imu" name="leo_imu_sensor">
+        <update_rate>100</update_rate>
+        <visualize>true</visualize>
+        <topic>imu/data_raw</topic>
+        <always_on>1</always_on>
+        <ignition_frame_id>imu_frame</ignition_frame_id>
+      </sensor>
+    </gazebo>
+    <gazebo>
+      <plugin
+        filename="libignition-gazebo-diff-drive-system.so"
+        name="ignition::gazebo::systems::DiffDrive">
+        <left_joint>wheel_FL_joint</left_joint>
+        <right_joint>wheel_FR_joint</right_joint>
+        <left_joint>wheel_RL_joint</left_joint>
+        <right_joint>wheel_RR_joint</right_joint>
+        <wheel_separation>0.358</wheel_separation>
+        <wheel_radius>0.0625</wheel_radius>
+        <frame_id>odom</frame_id>
+        <child_frame_id>base_footprint</child_frame_id>
+        <odom_publish_frequency>20</odom_publish_frequency>
+        <topic>cmd_vel</topic>
+        <odom_topic>odom</odom_topic>
+        <tf_topic>tf</tf_topic>
+        <max_linear_acceleration>2.5</max_linear_acceleration>
+        <max_angular_acceleration>3</max_angular_acceleration>
+        <min_linear_acceleration>-2.5</min_linear_acceleration>
+        <min_angular_acceleration>-3</min_angular_acceleration>
+      </plugin>
+    </gazebo>
+     <!-- lidar -->
     <gazebo reference="rplidar_link">
         <sensor type="gpu_lidar" name="generic_lidar_sensor">
-          <topic>${link_prefix}scan</topic>
+          <topic>scan</topic>
           <frame_id>rplidar_link</frame_id>
           <ignition_frame_id>rplidar_link</ignition_frame_id>
@@ -476,5 +559,5 @@
             </scan>
             <range>
-              <min>0.10</min>
+              <min>0.20</min>
               <max>10.0</max>
               <resolution>0.03</resolution>
@@ -495,73 +578,18 @@
         </plugin>
     </gazebo>
-    <!-- rocker differential -->
-    <gazebo>
-      <plugin name="leo_gz::DifferentialSystem" filename="libleo_gz_differential_plugin.so">
-        <jointA>rocker_L_joint</jointA>
-        <jointB>rocker_R_joint</jointB>
-        <forceConstant>100.0</forceConstant>
-      </plugin>
-    </gazebo>
-    <gazebo>
-      <plugin
-        filename="ignition-gazebo-joint-state-publisher-system"
-        name="ignition::gazebo::systems::JointStatePublisher">
-        <topic>${link_prefix}joint_states</topic>
-      </plugin>
-      <plugin filename="libignition-gazebo-imu-system.so"
-        name="ignition::gazebo::systems::Imu">
-      </plugin>
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