Commit message: Updated for integration with real life rover
Use real life rover: use_sim_time:=false

File: t1_rover/urdf/macros.xacro (robot description, xacro)
@@ -155,5 +155,5 @@
     <link name="camera_optical_frame"/>
     <link name="imu_frame"/>
-    <link name="laser_frame"/>
+    <link name="laser"/>
     <!--LIDAR LINK-->
     <link name="rplidar_link">
@@ -302,5 +302,5 @@
       <origin xyz="0 0 0.0368" rpy="0 0 ${pi}"/>
       <parent link="rplidar_link"/>
-      <child link="laser_frame"/>
+      <child link="laser"/>
     </joint>
   </xacro:macro>

Commit message: Add files via upload

File: t1_rover/urdf/macros.xacro (robot description, xacro)
@@ -155,38 +155,37 @@
     <link name="camera_optical_frame"/>
     <link name="imu_frame"/>
-    <link name="laser"/>
     <!--LIDAR LINK-->
-    <link name="rplidar_link">
-    <visual>
-      <origin xyz="0 0 0.003"/>
-      <geometry>
-        <box size="0.079 0.086 0.006"/>
-      </geometry>
-      <material name="support">
-        <color rgba="0.5 0.5 0.5 1.0"/>
-      </material>
-    </visual>
-    <visual>
-      <origin xyz="0 0 0.023"/>
-      <geometry>
-        <cylinder radius="0.038" length="0.04"/>
-      </geometry>
-      <material name="lidar">
-        <color rgba="1.0 0.0 0.0 0.7"/>
-      </material>
-    </visual>
-    <collision>
-      <origin xyz="0 0 0.003"/>
-      <geometry>
-        <box size="0.079 0.086 0.006"/>
-      </geometry>
-    </collision>
-    <collision>
-      <origin xyz="0 0 0.023"/>
-      <geometry>
-        <cylinder radius="0.038" length="0.04"/>
-      </geometry>
-    </collision>
-  </link>
+    <link name="laser">
+      <visual>
+        <origin xyz="0 0 0.003"/>
+        <geometry>
+          <box size="0.079 0.086 0.006"/>
+        </geometry>
+        <material name="support">
+          <color rgba="0.5 0.5 0.5 1.0"/>
+        </material>
+      </visual>
+      <visual>
+        <origin xyz="0 0 0.023"/>
+        <geometry>
+          <cylinder radius="0.038" length="0.04"/>
+        </geometry>
+        <material name="lidar">
+          <color rgba="1.0 0.0 0.0 0.7"/>
+        </material>
+      </visual>
+      <collision>
+        <origin xyz="0 0 0.003"/>
+        <geometry>
+          <box size="0.079 0.086 0.006"/>
+        </geometry>
+      </collision>
+      <collision>
+        <origin xyz="0 0 0.023"/>
+        <geometry>
+          <cylinder radius="0.038" length="0.04"/>
+        </geometry>
+      </collision>
+    </link>
     <!-- JOINTS -->
     <xacro:if value="${footprint_link}">
@@ -297,9 +296,4 @@
       <origin xyz="0.0775 0 0"/>
       <parent link="base_link"/>
-      <child link="rplidar_link"/>
-    </joint>
-    <joint name="laser_joint" type="fixed">
-      <origin xyz="0 0 0.0368" rpy="0 0 ${pi}"/>
-      <parent link="rplidar_link"/>
       <child link="laser"/>
     </joint>
@@ -543,9 +537,9 @@
     </gazebo>
      <!-- lidar -->
-    <gazebo reference="rplidar_link">
+    <gazebo reference="laser">
         <sensor type="gpu_lidar" name="generic_lidar_sensor">
           <topic>scan</topic>
-          <frame_id>rplidar_link</frame_id>
-          <ignition_frame_id>rplidar_link</ignition_frame_id>
+          <frame_id>laser</frame_id>
+          <ignition_frame_id>laser</ignition_frame_id>
           <update_rate>10.0</update_rate>
           <ray>
